Commit message: iris & typhoon models: enable lock-stepping
it's set to 2 because gazebo runs with 500Hz and the PX4 simulator
outputs mavlink control messages with 250Hz

File: models/rotors_description/urdf/component_snippets.xacro (robot description, xacro)
@@ -119,5 +119,5 @@
   </xacro:macro>
   <!-- Macro to add the mavlink interface. -->
-  <xacro:macro name="mavlink_interface_macro" params="namespace imu_sub_topic mavlink_addr mavlink_udp_port">
+  <xacro:macro name="mavlink_interface_macro" params="namespace imu_sub_topic mavlink_addr mavlink_udp_port sim_steps_per_mavlink_controls_msg">
     <gazebo>
       <plugin name="mavlink_interface" filename="librotors_gazebo_mavlink_interface.so">
@@ -126,4 +126,5 @@
         <mavlink_addr>$(arg mavlink_addr)</mavlink_addr>
         <mavlink_udp_port>$(arg mavlink_udp_port)</mavlink_udp_port>
+        <sim_steps_per_mavlink_controls_msg>$(arg sim_steps_per_mavlink_controls_msg)</sim_steps_per_mavlink_controls_msg>
         <motorSpeedCommandPubTopic>/gazebo/command/motor_speed</motorSpeedCommandPubTopic>
         <control_channels>

File: models/rotors_description/urdf/iris_base.xacro (robot description, xacro)
@@ -7,4 +7,5 @@
   <xacro:arg name='mavlink_udp_port' default='14560' />
   <xacro:arg name='visual_material' default='DarkGrey' />
+  <xacro:arg name='sim_steps_per_mavlink_controls_msg' default='2' />
   <!-- macros for gazebo plugins, sensors -->
   <xacro:include filename="$(arg rotors_description_dir)/urdf/component_snippets.xacro" />
@@ -18,4 +19,5 @@
     mavlink_addr="INADDR_ANY"
     mavlink_udp_port="14560"
+    sim_steps_per_mavlink_controls_msg="2"
     >
   </xacro:mavlink_interface_macro>
